File: nano/led-dimmer-4ch/KiCad/led-dimmer-4ch/led-dimmer-4ch.kicad_sch (KiCad schematic)
At the start: 32 parts, among them J1 Screw_Terminal_01x02, J2 Screw_Terminal_01x08, U1 LM2596S-5

Commit message: build(led-dimmer-4ch): assign hand-solderable SMD footprints to passives
- What: assigned KiCad footprints to R1-R4 and C1/C4/C5/C6 in led-dimmer-4ch.kicad_sch (previously unassigned).
- Why: the board needs a concrete footprint per part before it can be fabricated.
- How: 0805 hand-solder variants (Resistor_SMD:R_0805_2012Metric_..._HandSolder, Capacitor_SMD:C_0805_2012Metric_..._HandSolder) — larger pads than the standard 0805 footprint, sized for iron assembly rather than reflow.
- Benefit: the schematic now specifies parts that can be hand-assembled, consistent with this being a hobby build rather than a production run.
Parts:
- C1, C4, C5, C6: footprint (none) -> Capacitor_SMD:C_0805_2012Metric_Pad1.18x1.45mm_HandSolder
- R1, R2, R4: footprint (none) -> Resistor_SMD:R_0805_2012Metric_Pad1.20x1.40mm_HandSolder
Changed lines of the file:
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@@
 			)
 		)
-		(property "Footprint" ""
+		(property "Footprint" "Resistor_SMD:R_0805_2012Metric_Pad1.20x1.40mm_HandSolder"
 			(at 152.654 75.184 90)
 			(hide yes)
@@
 			)
 		)
-		(property "Footprint" ""
+		(property "Footprint" "Resistor_SMD:R_0805_2012Metric_Pad1.20x1.40mm_HandSolder"
 			(at 216.154 75.184 90)
 			(hide yes)
@@
 			)
 		)
-		(property "Footprint" ""
+		(property "Footprint" "Capacitor_SMD:C_0805_2012Metric_Pad1.18x1.45mm_HandSolder"
 			(at 130.5052 86.36 0)
 			(hide yes)
@@
 			)
 		)
-		(property "Footprint" ""
+		(property "Footprint" "Capacitor_SMD:C_0805_2012Metric_Pad1.18x1.45mm_HandSolder"
 			(at 130.5052 35.56 0)
 			(hide yes)
@@
 			)
 		)
-		(property "Footprint" ""
+		(property "Footprint" "Capacitor_SMD:C_0805_2012Metric_Pad1.18x1.45mm_HandSolder"
 			(at 194.0052 35.56 0)
 			(hide yes)
@@
 			)
 		)
-		(property "Footprint" ""
+		(property "Footprint" "Capacitor_SMD:C_0805_2012Metric_Pad1.18x1.45mm_HandSolder"
 			(at 194.0052 86.36 0)
 			(hide yes)
@@
 			)
 		)
-		(property "Footprint" ""
+		(property "Footprint" "Resistor_SMD:R_0805_2012Metric_Pad1.20x1.40mm_HandSolder"
 			(at 152.654 24.384 90)
 			(hide yes)
