File: arduino-nano/led-dimmer-4ch/hw/kicad/led-dimmer-4ch.kicad_sch (KiCad schematic)
At the start: 45 parts, among them J1 Screw_Terminal_01x02, J2 Screw_Terminal_01x04, J3 Screw_Terminal_01x04, J4 Screw_Terminal_01x04, J5 Screw_Terminal_01x04, U1 PT4115, U2 PT4115, U3 PT4115, U4 PT4115, U5 AP63205WU

Commit message: refactor(arduino-nano): move both boards into symmetric fw/ and hw/ packages
- What: moves each KiCad project to hw/kicad/, datasheets to hw/datasheets/, the microwave enclosure DXF to hw/mech/enclosure-template.dxf, and the microwave firmware into fw/, and deletes the stale microwave.csv, microwave.net, and toy-microwave.pdf exports.
- Why: the two boards used different layouts, and generated files sat beside the KiCad sources with no way to rebuild them.
- How: writes MPN, Manufacturer, Digi-Key, Mouser, and LCSC fields from parts.csv into every schematic symbol and PCB footprint, marks the Nano and MX switches Exclude from BOM per the part policy, gives the dimmer a rev 1 title block, points its sym-lib-table at kicad/embedded.kicad_sym, and adds one ../ to the microwave lib_deps.
- Benefit: both boards share one layout, each schematic carries its own purchasing data, and the microwave firmware still builds with 31 of 31 native tests passing.
Parts:
- A1: now left out of the parts list
- C1, C2, C3, C4: Digi-Key (none) -> 399-C1210C475K5RACAUTO7210CT-ND; MPN (none) -> C1210C475K5RACAUTO7210; Manufacturer (none) -> KEMET; Mouser (none) -> 80-C1210C475K5RAULR
- C10, C11, C12, C6, C9: Digi-Key (none) -> 399-12977-1-ND; MPN (none) -> C0805C104M5RACAUTO; Manufacturer (none) -> KEMET; Mouser (none) -> 80-C0805C104M5RAUTO
- C5: Digi-Key (none) -> 587-TMK325AB7106MMHPRCT-ND; MPN (none) -> TMK325AB7106MMHPR; Manufacturer (none) -> Taiyo Yuden; Mouser (none) -> 963-TMK325AB7106MMPR
- C7, C8: Digi-Key (none) -> 1276-3373-1-ND; MPN (none) -> CL32A226MAJNNNE; Manufacturer (none) -> Samsung; Mouser (none) -> 187-CL32A226MAJNNNE
- D1, D2, D3, D4, D5: Digi-Key (none) -> SS14-E3/61TGICT-ND; MPN (none) -> SS14-E3/61T; Manufacturer (none) -> Vishay; Mouser (none) -> 625-SS14-E3
- J1: Digi-Key (none) -> 277-1263-ND; MPN (none) -> 1715721; Manufacturer (none) -> Phoenix Contact; Mouser (none) -> 651-1715721
- J2, J3, J4, J5: Digi-Key (none) -> 277-1265-ND; MPN (none) -> 1715747; Manufacturer (none) -> Phoenix Contact; Mouser (none) -> 651-1715747
- L1, L2, L3, L4: MPN (none) -> MSS1038-104MLC; Manufacturer (none) -> Coilcraft; Mouser (none) -> 994-MSS1038-104MLC
- L5: Digi-Key (none) -> 490-LQH55DN4R7M03LCT-ND; MPN (none) -> LQH55DN4R7M03L; Manufacturer (none) -> Murata; Mouser (none) -> 81-LQH55DN4R7M03L
- R1, R2, R3, R4: Digi-Key (none) -> 273-KDV08FR360ETCT-ND; MPN (none) -> KDV08FR360ET; Manufacturer (none) -> Ohmite; Mouser (none) -> 588-KDV08FR360ET
- R5, R6, R7, R8: Digi-Key (none) -> 311-10.0KCRCT-ND; MPN (none) -> RC0805FR-0710KL; Manufacturer (none) -> Yageo; Mouser (none) -> 603-RC0805FR-0710KL
- U1, U2, U3, U4: Digi-Key (none) -> 4518-PT4115CT-ND; MPN (none) -> PT4115; Manufacturer (none) -> UMW
- U5: Digi-Key (none) -> AP63205WU-7DICT-ND; MPN (none) -> AP63205WU-7; Manufacturer (none) -> Diodes Inc; Mouser (none) -> 621-AP63205WU-7
Other:
- title: (none) -> 4-Channel LED Dimmer
