File: arduino-nano/toy-microwave-et6226m/hw/kicad/microwave.kicad_pcb (KiCad board)
At the start: 2 copper layers, 76.2 x 165.1 mm, 64 parts, among them J1 Screw_Terminal_01x04, J2 Screw_Terminal_01x04, Q2 AO3400A, U1 AP63205WU, U2 CC56-12SURKWA, U5 ET6226M

Commit message: feat(toy-microwave-et6226m): make J2 a grounded logic header with pull-downs
- What: reorders J2 to LIGHT, MOTOR, FAN, GND, moves CTRL_LIGHT to D10 and CTRL_BUZZER to D6, adds 10 kOhm pull-downs R11-R13 on the three control lines, and marks D13 no-connect.
- Why: J2 had no ground for off-board peripheral boards to reference, and the control lines floated while the Nano was in reset.
- How: replaced CTRL_MISC on pin 4 with GND, placed and routed R11-R13 as RC0805FR-0710KL, and kept outputs logic-level so each peripheral owns its driver and power.
- Benefit: any peripheral board can take its signals and ground from one connector and sees every line held low through reset, with ERC clean and 0 unconnected pads.
Parts:
- added R11: 10k, Resistor_SMD:R_0805_2012Metric_Pad1.20x1.40mm_HandSolder, B.Cu at (39.4, 182.2)
- added R12: 10k, Resistor_SMD:R_0805_2012Metric_Pad1.20x1.40mm_HandSolder, B.Cu at (36.8, 182.2)
- added R13: 10k, Resistor_SMD:R_0805_2012Metric_Pad1.20x1.40mm_HandSolder, B.Cu at (34.3, 182.2)
Connections:
- A1 pad 13: CTRL_BUZZER -> CTRL_LIGHT
- A1 pad 16: CTRL_LIGHT -> unconnected-(A1-D13-Pad16)
- A1 pad 9: CTRL_MISC -> CTRL_BUZZER
- J2 pad 1: CTRL_MOTOR -> CTRL_LIGHT
- J2 pad 2: CTRL_FAN -> CTRL_MOTOR
- J2 pad 3: CTRL_LIGHT -> CTRL_FAN
- J2 pad 4: CTRL_MISC -> GND
Routing:
- net CTRL_MISC: track 19.1 -> 0.00 mm
- net CTRL_BUZZER: track 154.1 -> 159.8 mm
- net CTRL_MOTOR: track 29.8 -> 25.6 mm
- net CTRL_LIGHT: track 32.2 -> 28.1 mm
- net CTRL_FAN: track 27.2 -> 25.4 mm
